Commit message: urdf update

File: apsara/urdf/arm.xacro (robot description, xacro)
@@ -220,5 +220,5 @@
       <inertial>
         <mass value="5" />
-        <origin rpy="0 0 0 " xyz="0 0 045" />
+        <origin rpy="0 0 0 " xyz="0 0 0.045" />
         <inertia ixx="170.667" ixy="0" ixz="0"
               iyy="170.667" iyz="0"
@@ -226,11 +226,11 @@
       </inertial>
       <collision>
-        <origin rpy="0 0 0 " xyz="0 0 045" />
-        <geometry>
-          <box size="0.1 0.1 0.1" />
-        </geometry>
-      </collision>
-      <visual>
-        <origin rpy="0 0 0 " xyz="0 0 045" />
+        <origin rpy="0 0 0 " xyz="0 0 0.045" />
+        <geometry>
+          <box size="0.1 0.1 0.1" />
+        </geometry>
+      </collision>
+      <visual>
+        <origin rpy="0 0 0 " xyz="0 0 0.045" />
         <geometry>
           <box size="0.1 0.1 0.1" />

File: apsara/urdf/links_joints.xacro (robot description, xacro)
@@ -62,5 +62,5 @@
     </link>
   </xacro:macro>
-  <xacro:macro name="m_link_mesh" params="name origin_xyz origin_rpy meshfile1 mass ixx ixy ixz iyy iyz izz">
+  <xacro:macro name="m_link_mesh" params="name origin_xyz origin_rpy meshfile meshscale mass ixx ixy ixz iyy iyz izz">
     <link name="${name}">
       <inertial>
@@ -72,5 +72,5 @@
         <origin rpy="${origin_rpy}" xyz="${origin_xyz}" />
         <geometry>
-          <mesh filename="${meshfile1}" scale="0.001 0.001 0.001"/>
+          <mesh filename="${meshfile}" scale="${meshscale}"/>
         </geometry>
       </collision>
@@ -78,6 +78,7 @@
         <origin rpy="${origin_rpy}" xyz="${origin_xyz}" />
         <geometry>
-          <mesh filename="${meshfile1}" scale="0.001 0.001 0.001"/>
+          <mesh filename="${meshfile}" scale="${meshscale}"/>
         </geometry>
+        <material name="light_black"/>
       </visual>
     </link>

File: apsara/urdf/mrm.xacro (robot description, xacro)
@@ -24,6 +24,6 @@
               iyy="13.235" iyz="0"
               izz="9.655"
-              meshfile1="package://apsara/meshes/link01.stl"
-             />
+              meshfile="package://apsara/meshes/link01.stl"
+              meshscale="0.001 0.001 0.001" />
   <m_joint name="${link_01_name}__${link_02_name}" type="revolute"
            axis_xyz="0 1 0"
@@ -37,6 +37,6 @@
               iyy="13.235" iyz="0"
               izz="9.655"
-              meshfile1="package://apsara/meshes/link12.stl"
-             />
+              meshfile="package://apsara/meshes/link12.stl"
+              meshscale="0.001 0.001 0.001" />
   <m_joint name="${link_02_name}__${link_03_name}" type="revolute"
            axis_xyz="0 1 0"
@@ -50,6 +50,6 @@
               iyy="13.235" iyz="0"
               izz="9.655"
-              meshfile1="package://apsara/meshes/link23.stl"
-               />
+              meshfile="package://apsara/meshes/link23.stl"
+              meshscale="0.001 0.001 0.001" />
   <m_joint name="${link_03_name}__${link_04_name}" type="revolute"
            axis_xyz="0 0 1"
@@ -63,22 +63,11 @@
               iyy="13.235" iyz="0"
               izz="9.655"
-              meshfile1="package://apsara/meshes/link34.stl"
-               />
+              meshfile="package://apsara/meshes/link34.stl"
+              meshscale="0.001 0.001 0.001" />
   <m_joint name="${link_04_name}__${link_05_name}" type="revolute"
            axis_xyz="0 1 0"
-             meshfile1="package://apsara/meshes/link45.stl"
-               />
-  <m_joint name="${link_05_name}__${link_06_name}" type="revolute"
-           axis_xyz="0 0 1"
-           origin_rpy="0 0 0" origin_xyz="0 0 0.1628"
-           parent="link_05" child="link_06"
-           limit_e="1000" limit_l="-3.14" limit_u="3.14" limit_v="0.5" />
-  <m_link_box name="${link_06_name}"
-              origin_rpy="0 0 0" origin_xyz="0 0 0.045"
-              mass="1024"
-              ixx="170.667" ixy="0" ixz="0"
-              iyy="170.667" iyz="0"
-              izz="170.667"
-              size="0.1 0.1 0.1" />imit_e="1000" limit_l="-2.24" limit_u="2.24" limit_v="0.5" />
+           origin_rpy="0 0 0" origin_xyz="0 0 0.1493"
+           parent="link_04" child="link_05"
+           limit_e="1000" limit_l="-2.24" limit_u="2.24" limit_v="0.5" />
   <m_link_mesh name="${link_05_name}"
               origin_rpy="0 0 0" origin_xyz="0 0 -0.7085"
@@ -87,5 +76,6 @@
               iyy="13.235" iyz="0"
               izz="9.655"
-              meshfile1="package://apsara/meshes/link45.stl" />
+              meshfile="package://apsara/meshes/link45.stl"
+              meshscale="0.001 0.001 0.001" />
   <m_joint name="${link_05_name}__${link_06_name}" type="revolute"
            axis_xyz="0 0 1"
@@ -100,5 +90,5 @@
               izz="170.667"
               size="0.1 0.1 0.1" />
-   END - Robot description -->
+  <!-- END - Robot description -->
   <gazebo>
     <plugin name="gazebo_ros_control" filename="libgazebo_ros_control.so">

Commit message: realsense

File: apsara/urdf/arm.xacro (robot description, xacro)
@@ -1,4 +1,20 @@
 <?xml version="1.0" ?>
 <robot name="arm" xmlns:xacro="http://www.ros.org/wiki/xacro">
+  <xacro:include filename="$(find apsara)/urdf/1_d435.urdf.xacro" />
+  <xacro:include filename="$(find apsara)/urdf/2_d435.urdf.xacro" />
+     <!-- world will be root link-->
+  <link name="world" />
+  <joint name="world_joint" type="fixed">
+    <parent link="world" />
+    <child link = "pole_link" />
+    <origin xyz="0.0 0.0 0.1" rpy="0.0 0.0 0.0" />
+  </joint>
+  <link name="pole_link">
+    <visual>
+      <geometry>
+        <cylinder length="1.5" radius="0.1"/>
+      </geometry>
+    </visual>
+  </link>
     <link name="base_link">
       <inertial>
@@ -20,4 +36,9 @@
       </visual>
     </link>
+   <joint name="pole_joint" type="fixed">
+      <parent link="pole_link" />
+      <child link="base_link" />
+      <origin xyz="0 0 0.75"/>
+    </joint>
     <link name="link_01">
       <inertial>
@@ -49,8 +70,8 @@
       <type>transmission_interface/SimpleTransmission</type>
       <joint name="base_link__link_01">
-        <hardwareInterface>hardware_interface/EffortJointInterface</hardwareInterface>
+        <hardwareInterface>hardware_interface/PositionJointInterface</hardwareInterface>
       </joint>
       <actuator name="motor_base_link__link_01">
-        <hardwareInterface>hardware_interface/EffortJointInterface</hardwareInterface>
+        <hardwareInterface>hardware_interface/PositionJointInterface</hardwareInterface>
         <mechanicalReduction>1</mechanicalReduction>
       </actuator>
@@ -66,8 +87,8 @@
       <type>transmission_interface/SimpleTransmission</type>
       <joint name="link_01__link_02">
-        <hardwareInterface>hardware_interface/EffortJointInterface</hardwareInterface>
+        <hardwareInterface>hardware_interface/PositionJointInterface</hardwareInterface>
       </joint>
       <actuator name="motor_link_01__link_02">
-        <hardwareInterface>hardware_interface/EffortJointInterface</hardwareInterface>
+        <hardwareInterface>hardware_interface/PositionJointInterface</hardwareInterface>
         <mechanicalReduction>1</mechanicalReduction>
       </actuator>
@@ -102,8 +123,8 @@
       <type>transmission_interface/SimpleTransmission</type>
       <joint name="link_02__link_03">
-        <hardwareInterface>hardware_interface/EffortJointInterface</hardwareInterface>
+        <hardwareInterface>hardware_interface/PositionJointInterface</hardwareInterface>
       </joint>
       <actuator name="motor_link_02__link_03">
-        <hardwareInterface>hardware_interface/EffortJointInterface</hardwareInterface>
+        <hardwareInterface>hardware_interface/PositionJointInterface</hardwareInterface>
         <mechanicalReduction>1</mechanicalReduction>
       </actuator>
@@ -138,8 +159,8 @@
       <type>transmission_interface/SimpleTransmission</type>
       <joint name="link_03__link_04">
-        <hardwareInterface>hardware_interface/EffortJointInterface</hardwareInterface>
+        <hardwareInterface>hardware_interface/PositionJointInterface</hardwareInterface>
       </joint>
       <actuator name="motor_link_03__link_04">
-        <hardwareInterface>hardware_interface/EffortJointInterface</hardwareInterface>
+        <hardwareInterface>hardware_interface/PositionJointInterface</hardwareInterface>
         <mechanicalReduction>1</mechanicalReduction>
       </actuator>
@@ -174,8 +195,8 @@
       <type>transmission_interface/SimpleTransmission</type>
       <joint name="link_04__link_05">
-        <hardwareInterface>hardware_interface/EffortJointInterface</hardwareInterface>
+        <hardwareInterface>hardware_interface/PositionJointInterface</hardwareInterface>
       </joint>
       <actuator name="motor_link_04__link_05">
-        <hardwareInterface>hardware_interface/EffortJointInterface</hardwareInterface>
+        <hardwareInterface>hardware_interface/PositionJointInterface</hardwareInterface>
         <mechanicalReduction>1</mechanicalReduction>
       </actuator>
@@ -210,8 +231,8 @@
       <type>transmission_interface/SimpleTransmission</type>
       <joint name="link_05__link_06">
-        <hardwareInterface>hardware_interface/EffortJointInterface</hardwareInterface>
+        <hardwareInterface>hardware_interface/PositionJointInterface</hardwareInterface>
       </joint>
       <actuator name="motor_link_05__link_06">
-        <hardwareInterface>hardware_interface/EffortJointInterface</hardwareInterface>
+        <hardwareInterface>hardware_interface/PositionJointInterface</hardwareInterface>
         <mechanicalReduction>1</mechanicalReduction>
       </actuator>
@@ -238,3 +259,37 @@
       </visual>
     </link>
+  <gazebo>
+    <plugin name="gazebo_ros_control" filename="libgazebo_ros_control.so">
+    </plugin>
+  </gazebo>
+  <link name="cam_pole_link">
+    <visual>
+      <geometry>
+        <cylinder length="1" radius="0.03"/>
+      </geometry>
+    </visual>
+  </link>
+<joint name="cam_pole_joint" type="fixed">
+      <parent link="world" />
+      <child link="cam_pole_link" />
+      <origin xyz="0 2 0.5"/>
+</joint>
+<sensor1_d435 parent="cam_pole_link">
+    <origin xyz="0.0 0.0 0.5" rpy="0 0 1.5708"/>
+</sensor1_d435>
+<link name="cam_pole_link2">
+    <visual>
+      <geometry>
+        <cylinder length="1" radius="0.03"/>
+      </geometry>
+    </visual>
+</link>
+<joint name="cam_pole_joint2" type="fixed">
+      <parent link="world" />
+      <child link="cam_pole_link2" />
+      <origin xyz="0 -2 0.5"/>
+</joint>
+<sensor2_d435 parent="cam_pole_link2">
+    <origin xyz="0.0 0.0 0.5" rpy="0 0 -1.5708"/>
+</sensor2_d435>
 </robot>

Commit message: realsense edit

File: apsara/urdf/arm.xacro (robot description, xacro)
@@ -276,5 +276,5 @@
 </joint>
 <sensor1_d435 parent="cam_pole_link">
-    <origin xyz="0.0 0.0 0.5" rpy="0 0 1.5708"/>
+    <origin xyz="0.0 0.0 0.5" rpy="0 0 -1.5708"/>
 </sensor1_d435>
 <link name="cam_pole_link2">
@@ -291,5 +291,5 @@
 </joint>
 <sensor2_d435 parent="cam_pole_link2">
-    <origin xyz="0.0 0.0 0.5" rpy="0 0 -1.5708"/>
+    <origin xyz="0.0 0.0 0.5" rpy="0 0 1.5708"/>
 </sensor2_d435>
 </robot>
